File: ANGEL_001/001_PCB/001_PCB.kicad_sch (KiCad schematic)
At the start: 67 parts, among them J1 USB_C_Receptacle_USB2.0_14P, SW1 SW_Push_1P1T-SH_NO_CK_KMR2xxG, SW2 SW_Push_1P1T-SH_NO_CK_KMR2xxG, U1 ESP32-MINI-1, U10 MSA311, U12 TPS62172DSG, U13 BQ24072RGT, U2 STM32H750VBTx, U3 PCM3060, U4 IS25LP032D-JNLE, U5 MCP9700x-HTT, U6 USBLC6-2SC6, U7 BQ27220, U8 LP2985-5.0, U9 CAP1188, Y2 16MHz

Commit message: PCB work + speaker testing
Parts:
- removed C11: 4.7uF, symbol Device:C_Small
- removed C12: 1uF, symbol Device:C_Small
- removed D3: B120-E3, Diode_SMD:D_SMA, symbol Diode:B120-E3
- removed J1: USB_C_Receptacle_USB2.0_14P, symbol Connector:USB_C_Receptacle_USB2.0_14P
- removed R12: 0.01, symbol Device:R_Small
- removed R13, R14: 10k, symbol Device:R_Small
- removed R15, R16: 5k1, symbol Device:R_Small
- removed U1: ESP32-MINI-1, PCM_Espressif:ESP32-MINI-1, symbol PCM_Espressif:ESP32-MINI-1
- removed U7: BQ27220, Package_BGA:Texas_DSBGA-9_1.62x1.58mm_Layout3x3_P0.5mm, symbol Battery_Management:BQ27220
- added C1, C15, C16, C20, C22, C32, C40, C42: 100nF, Capacitor_SMD:C_0402_1005Metric_Pad0.74x0.62mm_HandSolder, symbol Device:C_Small
- added C17, C18, C19, C24, C4, C41: 10uF, Capacitor_SMD:C_0805_2012Metric_Pad1.18x1.45mm_HandSolder, symbol Device:C_Small
- added C21: 1uF, Capacitor_SMD:C_0603_1608Metric_Pad1.08x0.95mm_HandSolder, symbol Device:C_Small
- added C27: 10nF, Capacitor_SMD:C_0402_1005Metric_Pad0.74x0.62mm_HandSolder, symbol Device:C_Small
- added C28: 2.2uF, Capacitor_SMD:C_0603_1608Metric_Pad1.08x0.95mm_HandSolder, symbol Device:C_Small
- added C29, C30: 220pF, Capacitor_SMD:C_0402_1005Metric_Pad0.74x0.62mm_HandSolder, symbol Device:C_Small
- added D3: D, Diode_SMD:D_SOD-123, symbol Device:D
- added FB1, FB2, FB3: FerriteBead_Small, Inductor_SMD:L_0402_1005Metric_Pad0.77x0.64mm_HandSolder, symbol Device:FerriteBead_Small
- added J1: USB_B_Micro, Connector_USB:USB_Micro-B_Amphenol_10118193-0001LF_Horizontal, symbol Connector:USB_B_Micro
- added J3: AudioJack3_SwitchT, Connector_Audio:Jack_3.5mm_CUI_SJ-3524-SMT_Horizontal, symbol Connector_Audio:AudioJack3_SwitchT
- added LS1: Speaker, TerminalBlock:TerminalBlock_MaiXu_MX126-5.0-02P_1x02_P5.00mm, symbol Device:Speaker
- added R18, R21, R6, R7: 10k, Resistor_SMD:R_0402_1005Metric_Pad0.72x0.64mm_HandSolder, symbol Device:R_Small
- added R19: 150k, Resistor_SMD:R_0402_1005Metric_Pad0.72x0.64mm_HandSolder, symbol Device:R_Small
- added R20: 220k, Resistor_SMD:R_0402_1005Metric_Pad0.72x0.64mm_HandSolder, symbol Device:R_Small
- added R5: 5R1, Resistor_SMD:R_0402_1005Metric_Pad0.72x0.64mm_HandSolder, symbol Device:R_Small
- added RV1, RV2, RV3, RV4, RV5, RV6: 50k Trim, Potentiometer_SMD:Potentiometer_Bourns_TC33X_Vertical, symbol Device:R_Potentiometer_Trim
- added U4: PAM8302AAS, Package_SO:MSOP-8_3x3mm_P0.65mm, symbol Amplifier_Audio:PAM8302AAS
- BT1: footprint (none) -> Connector_JST:JST_PH_S2B-PH-SM4-TB_1x02-1MP_P2.00mm_Horizontal
- C10: renamed from C5; footprint (none) -> Capacitor_SMD:C_0402_1005Metric_Pad0.74x0.62mm_HandSolder
- C11: renamed from C1; footprint (none) -> Capacitor_SMD:C_0603_1608Metric_Pad1.08x0.95mm_HandSolder
- C12: renamed from C4; footprint (none) -> Capacitor_SMD:C_0402_1005Metric_Pad0.74x0.62mm_HandSolder
- C13: renamed from C2; footprint (none) -> Capacitor_SMD:C_0603_1608Metric_Pad1.08x0.95mm_HandSolder
- C14: renamed from C3; footprint (none) -> Capacitor_SMD:C_0603_1608Metric_Pad1.08x0.95mm_HandSolder
- C2: renamed from C8; footprint (none) -> Capacitor_SMD:C_0402_1005Metric_Pad0.74x0.62mm_HandSolder
- C25: renamed from C9; footprint (none) -> Capacitor_SMD:C_0603_1608Metric_Pad1.08x0.95mm_HandSolder
- C26: renamed from C10; footprint (none) -> Capacitor_SMD:C_0402_1005Metric_Pad0.74x0.62mm_HandSolder
- C3: renamed from C13; footprint (none) -> Capacitor_SMD:C_0402_1005Metric_Pad0.74x0.62mm_HandSolder
- C31: renamed from C15; footprint (none) -> Capacitor_SMD:C_0805_2012Metric_Pad1.18x1.45mm_HandSolder
- C33: renamed from C16; footprint (none) -> Capacitor_SMD:C_0402_1005Metric_Pad0.74x0.62mm_HandSolder
- C34: renamed from C20; footprint (none) -> Capacitor_SMD:C_0805_2012Metric_Pad1.18x1.45mm_HandSolder
- C35: renamed from C17; footprint (none) -> Capacitor_SMD:C_0805_2012Metric_Pad1.18x1.45mm_HandSolder
- C36: renamed from C21; footprint (none) -> Capacitor_SMD:C_0805_2012Metric_Pad1.18x1.45mm_HandSolder
- C37: renamed from C18; footprint (none) -> Capacitor_SMD:C_1206_3216Metric_Pad1.33x1.80mm_HandSolder
- C38: renamed from C22; footprint (none) -> Capacitor_SMD:C_0805_2012Metric_Pad1.18x1.45mm_HandSolder
- C39: renamed from C19; footprint (none) -> Capacitor_SMD:C_1206_3216Metric_Pad1.33x1.80mm_HandSolder
- C5: renamed from C7; footprint (none) -> Capacitor_SMD:C_0402_1005Metric_Pad0.74x0.62mm_HandSolder
- C6: renamed from C27; footprint (none) -> Capacitor_SMD:C_0402_1005Metric_Pad0.74x0.62mm_HandSolder
- C7: renamed from C33; footprint (none) -> Capacitor_SMD:C_0603_1608Metric_Pad1.08x0.95mm_HandSolder
- C8: renamed from C14; footprint (none) -> Capacitor_SMD:C_0402_1005Metric_Pad0.74x0.62mm_HandSolder
- C9: renamed from C6; footprint (none) -> Capacitor_SMD:C_0402_1005Metric_Pad0.74x0.62mm_HandSolder
- D1, D2: footprint (none) -> LED_SMD:LED_0805_2012Metric_Pad1.15x1.40mm_HandSolder
- FB4: renamed from FB1; footprint (none) -> Inductor_SMD:L_0402_1005Metric_Pad0.77x0.64mm_HandSolder
- H1, H2: now left out of the parts list
- L1: footprint (none) -> Inductor_SMD:L_Murata_DFE201610P
- P1: renamed from R1; value FSR -> FSR_Pinky; footprint (none) -> Library:FSR; now left out of the parts list
- P2: renamed from R2; value FSR -> FSR_Ring; footprint (none) -> Library:FSR; now left out of the parts list
- P3: renamed from R3; value FSR -> FSR_Middle; footprint (none) -> Library:FSR; now left out of the parts list
- P4: renamed from R4; value FSR -> FSR_Index; footprint (none) -> Library:FSR; now left out of the parts list
- P5: renamed from R5; value FSR -> FSR_Thumb; footprint (none) -> Library:FSR; now left out of the parts list
- P6: renamed from R6; value FSR -> FSR_Palm; footprint (none) -> Library:FSR; now left out of the parts list
- R1: renamed from R9; footprint (none) -> Resistor_SMD:R_0402_1005Metric_Pad0.72x0.64mm_HandSolder
- R12: renamed from R17; footprint (none) -> Resistor_SMD:R_0402_1005Metric_Pad0.72x0.64mm_HandSolder
- R16: renamed from R11; footprint (none) -> Resistor_SMD:R_0402_1005Metric_Pad0.72x0.64mm_HandSolder
- R2: renamed from R10; footprint (none) -> Resistor_SMD:R_0402_1005Metric_Pad0.72x0.64mm_HandSolder
- R3: renamed from R7; footprint (none) -> Resistor_SMD:R_0402_1005Metric_Pad0.72x0.64mm_HandSolder
- R4: renamed from R8; footprint (none) -> Resistor_SMD:R_0402_1005Metric_Pad0.72x0.64mm_HandSolder
- R8: renamed from R19; footprint (none) -> Resistor_SMD:R_0402_1005Metric_Pad0.72x0.64mm_HandSolder
- R9: renamed from R18; footprint (none) -> Resistor_SMD:R_0402_1005Metric_Pad0.72x0.64mm_HandSolder
- renumbered U3 to U1, U6 to U10, U9 to U11, U8 to U3, U4 to U5, U12 to U6, U13 to U7, U5 to U8, U10 to U9, Y2 to Y1
Connections:
- net PGND is gone; now on net GND: BT1.2 (-)
- net +3.3V: now also U1.1 (MC/SCL/FMT), U1.27 (~{MS}/AD/IFMD), U1.7 (V_{DD}), U11.23 (VDD), U5.8 (VCC), U9.7 (VDD), C1.1, C32.1, C4.1, C40.1, C41.1, C42.1, R18.1, R20.1, R21.1, R6.1, R7.1
- net +3.3VA: now also P1.1, P2.1, P3.1, P4.1, P5.1, P6.1, U8.1 (V_{DD})
- net GND: now also U1.16 (SGND), U1.22 (AGND2), U1.23 (AGND1), U1.8 (DGND), U11.10 (LED6), U11.11 (LED7), U11.12 (LED8), U11.24 (RESET), U11.25 (GND), U11.5 (LED1), U11.6 (LED2), U11.7 (LED3), U11.8 (LED4), U11.9 (LED5), U3.2 (GND), U5.4 (GND), U8.3 (GND), U9.4 (GND), U9.8 (GND), U9.9 (GND), C1.2, C15.2, C16.2, C17.2, C18.2, C19.2, C20.2, C21.2, C24.2, C27.2, C28.2, C29.2, C30.2, C32.2, C4.2, C40.2, C41.2, C42.2, J1.5 (GND), J3.S, R19.2, RV1.2, RV2.2, RV3.2, RV4.2, RV5.2, RV6.2, U4.4 (IN-), U4.7 (GND)
- net USB_DM: now also U10.4 (I/O2), U2.70 (PA11); no longer U10.6 (I/O1), U2.53 (PB14)
- net USB_DM_IN: now also U10.3 (I/O2), J1.2 (D-); no longer U10.1 (I/O1)
- net USB_DP: now also U10.6 (I/O1), U2.71 (PA12); no longer U10.4 (I/O2), U2.54 (PB15)
- net USB_DP_IN: now also U10.1 (I/O1), J1.3 (D+); no longer U10.3 (I/O2)
- net VBUS: now also J1.1 (VBUS)
- net VCHG: no longer C38.1, U7.10 (OUT), U7.11 (OUT)
- net QSPI_NCS: now reaches U5.1 (~{CS})
- net QSPI_NCS: now also U2.79 (PC11)
- net QSPI_IO1: now reaches U5.2 (D1/DO)
- net QSPI_IO1: now also U2.38 (PE8)
- net QSPI_IO2: now reaches U5.3 (D2/~{WP})
- net QSPI_IO2: now also U2.39 (PE9)
- net QSPI_IO0: now reaches U5.5 (D0/DI)
- net QSPI_IO0: now also U2.37 (PE7)
- net QSPI_CLK: now reaches U5.6 (CLK)
- net QSPI_CLK: now also U2.36 (PB2)
- net QSPI_IO3: now reaches U5.7 (D3/~{HOLD})
- net QSPI_IO3: now also U2.40 (PE10)
- net FSR_6: now reaches P6.2
- net FSR_6: now also U2.25 (PA3), RV6.1
- net at U11.13 (ALERT#): now also R18.2
- net at U11.14 (ADDR_COMM): now also R19.1
- net I2C1_SDA: now reaches U11.3 (SDA/SPI_MISO)
- net I2C1_SDA: now also U2.46 (PB10), U9.12 (SCL), R7.2
- net I2C1_SCL: now reaches U11.4 (SCL/SPI_CLK)
- net I2C1_SCL: now also U2.47 (PB11), U9.2 (SDA), R6.2
- net at U3.1 (VIN): now also U3.3 (ON/~{OFF}), C19.1, C21.1, R5.2
- net at U3.4 (BP): now also C27.1
- net at U3.5 (VOUT): now also C28.1, FB3.1
- net at C31.1, C33.1, FB4.1: now also D3.1 (K)
- net FSR_1: now reaches P1.2
- net FSR_1: now also U2.15 (PC0), RV1.1
- net TEMP_SENS: now reaches U8.2 (V_{OUT})
- net TEMP_SENS: now also U2.28 (PA4)
- net FSR_3: now reaches P3.2
- net FSR_3: now also U2.22 (PA0), RV3.1
- net FSR_5: now reaches P5.2
- net FSR_5: now also U2.24 (PA2), RV5.1
- net FSR_2: now reaches P2.2
- net FSR_2: now also U2.16 (PC1), RV2.1
- net FSR_4: now reaches P4.2
- net FSR_4: now also U2.23 (PA1), RV4.1
- net SAI1_MCLK: now reaches U2.1 (PE2)
- net SAI1_MCLK: now also U1.6 (SCKI1), U1.9 (SCKI2)
- net SAI1_SD_B: now reaches U2.2 (PE3)
- net SAI1_SD_B: now also U1.3 (DOUT)
- net SAI1_FS: now reaches U2.3 (PE4)
- net SAI1_FS: now also U1.11 (LRCK2), U1.4 (LRCK1)
- net SAI1_SCK: now reaches U2.4 (PE5)
- net SAI1_SCK: now also U1.10 (BCK2), U1.5 (BCK1)
- net SAI1_SD_A: now reaches U2.5 (PE6)
- net SAI1_SD_A: now also U1.12 (DIN)
- net USB_ID: now reaches U2.69 (PA10)
- net USB_ID: now also J1.4 (ID)
- net CODEC_DEMP: now reaches U2.7 (PC13)
- net CODEC_DEMP: now also U1.2 (MD/SDA/DEMP)
- net CODEC_RST: now reaches U2.8 (PC14)
- net CODEC_RST: now also U1.15 (~{RST}), R21.2
- net AMP_SD: now reaches U2.9 (PC15)
- net AMP_SD: now also U4.1 (~{SD})
- net AUDIO_R: now reaches U1.18 (V_{OUT}R+)
- net AUDIO_R: now also J3.R
- net AUDIO_L: now reaches U1.20 (V_{OUT}L+)
- net AUDIO_L: now also J3.T
- net at U1.21 (V_{COM}): now also C16.1, C18.1
- net +5V: now reaches U1.24 (V_{CC})
- net +5V: now also C15.1, C17.1, C20.1, C24.1, FB3.2, U4.6 (VDD)
- net at U1.28 (MODE): now also R20.2
- new net: FB1.1, U4.5 (OUT+)
- new net: C29.1, FB1.2, LS1.1
- new net: C22.2, U4.3 (IN+)
- new net: FB2.1, U4.8 (OUT-)
- new net: C30.1, FB2.2, LS1.2
- new net AUDIO_L_SP: C22.1, J3.TN
- new net VIN: C38.1, D3.2 (A), R5.1, U7.10 (OUT), U7.11 (OUT)
- no-connect marks 3 -> 22
Other:
- note added: "AGND1 is ADC GND AGND2 is DAC GND"
- note added: "ANALOG SENSORS"
- note added: "AUDIO OUT"
- note added: "AUDIO POWER"
- note added: "BATTERY CHARGE"
- note added: "CODEC"
- note added: "CODEC_RST Open Drain Pull to GND"
- note added: "Fast charge set to 800mA Current limit set to 1.3 A"
- note added: "SENSORS"
- note added: "USB"
- note removed: "BATTERY MONITOR + CHARGE"
- moved on the sheet: BT1, C25, C26, C34, C35, C36, C37, C38, FB4, H1, H2, L1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

Commit message: PCB finalization + FSR design
Parts:
- added J2: Conn_02x06_Odd_Even, Connector_PinHeader_2.00mm:PinHeader_2x06_P2.00mm_Vertical, symbol Connector_Generic:Conn_02x06_Odd_Even
- added R16: 0, symbol Device:R_Small
- BT1, R12, U7: now not fitted; now left out of the parts list
- C14: value 4.7uF -> 10uF; footprint Capacitor_SMD:C_0603_1608Metric_Pad1.08x0.95mm_HandSolder -> Capacitor_SMD:C_0805_2012Metric_Pad1.18x1.45mm_HandSolder
- C31: renamed from C34; now not fitted; now left out of the parts list
- C35: renamed from C36; now not fitted; now left out of the parts list
- C37: renamed from C38; now not fitted; now left out of the parts list
- LS1: footprint TerminalBlock:TerminalBlock_MaiXu_MX126-5.0-02P_1x02_P5.00mm -> Connector_PinHeader_2.00mm:PinHeader_1x02_P2.00mm_Vertical
- P1: footprint Library:FSR -> Library:FSR_Pinky
- P2: footprint Library:FSR -> Library:FSR_Ring
- P3: footprint Library:FSR -> Library:FSR_Middle
- P4: footprint Library:FSR -> Library:FSR_Index
- P5: footprint Library:FSR -> Library:FSR_Thumb
- P6: footprint Library:FSR -> Library:FSR_Palm
- R10: renamed from R8; now not fitted; now left out of the parts list
- R11: renamed from R9; now not fitted; now left out of the parts list
- renumbered C21 to C20, C25 to C21, C26 to C22, C27 to C23, C20 to C24, C28 to C25, C22 to C26, C24 to C27, C31 to C28, C32 to C29, C33 to C30, C35 to C32, C29 to C33, C30 to C34, C37 to C36, C39 to C38, C42 to C39, FB3 to FB1, FB4 to FB2, FB1 to FB3, FB2 to FB4, J3 to J1, J1 to J3, R20 to R1, R16 to R13, R18 to R14, R19 to R15, R1 to R2, R21 to R3, R2 to R4, R3 to R5, R4 to R6, R5 to R7, R6 to R8, R7 to R9
Connections:
- net +3.3VA: now also J2.10 (Pin_10), J2.12 (Pin_12), J2.2 (Pin_2), J2.4 (Pin_4), J2.6 (Pin_6), J2.8 (Pin_8); no longer P1.1, P2.1, P3.1, P4.1, P5.1, P6.1
- net FSR_1: now also J2.1 (Pin_1); no longer P1.2
- net FSR_2: now also J2.3 (Pin_3); no longer P2.2
- net FSR_3: now also J2.5 (Pin_5); no longer P3.2
- net FSR_4: now also J2.7 (Pin_7); no longer P4.2
- net FSR_5: now also J2.9 (Pin_9); no longer P5.2
- net FSR_6: now also J2.11 (Pin_11); no longer P6.2
- net GND: no longer C1.2, C10.2, C11.2, C12.2, C13.2, C14.2, C15.2, C16.2, C17.2, C18.2, C19.2, C2.2, C20.2, C21.2, C22.2, C23.2, C24.2, C25.2, C27.2, C28.2, C29.2, C3.1, C30.2, C32.2, C33.2, C34.2, C36.2, C38.2, C39.2, C4.2, C40.2, C41.2, C5.2, C6.2, C7.2, C8.1, C9.2, D1.1 (K), D2.1 (K), J1.S, J3.5 (GND), R15.2, R6.2, RV1.2, RV2.2, RV3.2, RV4.2, RV5.2, RV6.2, SW1.1 (A), U1.16 (SGND), U1.22 (AGND2), U1.23 (AGND1), U1.8 (DGND), U10.2 (GND), U11.10 (LED6), U11.11 (LED7), U11.12 (LED8), U11.24 (RESET), U11.25 (GND), U11.5 (LED1), U11.6 (LED2), U11.7 (LED3), U11.8 (LED4), U11.9 (LED5), U2.10 (VSS), U2.19 (VSSA), U2.26 (VSS), U2.49 (VSS), U2.74 (VSS), U2.99 (VSS), U3.2 (GND), U4.4 (IN-), U4.7 (GND), U5.4 (GND), U6.1 (PGND), U6.4 (AGND), U6.5 (FB), U6.9 (PAD), U8.3 (GND), U9.4 (GND), U9.8 (GND), U9.9 (GND), Y1.2 (G), Y1.4 (G)
- net USB_DM: now also U10.6 (I/O1); no longer U10.4 (I/O2)
- net USB_DM_IN: now also U10.1 (I/O1); no longer U10.3 (I/O2)
- net USB_DP: now also U10.4 (I/O2); no longer U10.6 (I/O1)
- net USB_DP_IN: now also U10.3 (I/O2); no longer U10.1 (I/O1)
- net VBUS: no longer J3.1 (VBUS), U10.5 (VBUS)
- net VIN: now also J3.1 (VBUS), U10.5 (VBUS)
- new net GNDA: C15.2, C16.2, C17.2, C18.2, C19.2, C20.2, C21.2, C22.2, C23.2, C24.2, C25.2, C27.2, C33.2, C34.2, C38.2, J1.S, R16.2, RV1.2, RV2.2, RV3.2, RV4.2, RV5.2, RV6.2, U1.22 (AGND2), U1.23 (AGND1), U2.19 (VSSA), U3.2 (GND), U4.4 (IN-), U4.7 (GND), U8.3 (GND)
- new net GNDD: C1.2, C10.2, C11.2, C12.2, C13.2, C14.2, C2.2, C28.2, C29.2, C3.1, C30.2, C32.2, C36.2, C39.2, C4.2, C40.2, C41.2, C5.2, C6.2, C7.2, C8.1, C9.2, D1.1 (K), D2.1 (K), J3.5 (GND), R15.2, R16.1, R6.2, SW1.1 (A), U1.16 (SGND), U1.8 (DGND), U10.2 (GND), U11.10 (LED6), U11.11 (LED7), U11.12 (LED8), U11.24 (RESET), U11.25 (GND), U11.5 (LED1), U11.6 (LED2), U11.7 (LED3), U11.8 (LED4), U11.9 (LED5), U2.10 (VSS), U2.26 (VSS), U2.49 (VSS), U2.74 (VSS), U2.99 (VSS), U5.4 (GND), U6.1 (PGND), U6.4 (AGND), U6.5 (FB), U6.9 (PAD), U9.4 (GND), U9.8 (GND), U9.9 (GND), Y1.2 (G), Y1.4 (G)
- no-connect marks 22 -> 34
Other:
- note added: "Add test point pins to QSPI, i2s, i2c, power (all levels), gnd"
- moved on the sheet: P1, P2, P3, P4, P5, P6, RV1, RV2, RV3, RV4, RV5, RV6
